File: Hardware/weather-bit.brd (EAGLE design)
At the start: 68.6 x 63.5 mm, 41 parts, among them J1 EDGE-80PTH-RA, J2 RJ11, J3 RJ11, U1 BME280

Commit message: Updated Baord Layout, prepping for today's meeting
Parts:
- moved J6 45.8 mm to (39.4, 6.35), turned to 0 degrees
- moved J4 35.0 mm to (38.1, 15.2), turned to 0 degrees
- moved J7 28.0 mm to (24.1, 6.35), turned to 0 degrees
- moved R10 26.5 mm to (11.4, 22.9), turned to 270 degrees
- moved R8 26.5 mm to (8.89, 22.9)
- moved R1 24.8 mm to (29.2, 36.8)
- moved D4 22.5 mm to (41.9, 21.6)
- moved R2 20.3 mm to (35.6, 36.8)
- moved R3 19.1 mm to (40.6, 36.8)
- moved R11 18.8 mm to (45.1, 21.6)
- moved J5 16.6 mm to (22.9, 15.2), turned to 0 degrees
- moved D6 16.3 mm to (38.1, 21.6)
- moved J3 12.5 mm to (12.7, 10.2)
- moved J2 11.4 mm to (55.9, 10.2)
- moved D3 9.69 mm to (6.35, 22.9)
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Routing:
- net WSPEED: track 17.3 -> 53.5 mm, vias 0 -> 2
- net SOIL_DAT: track 21.2 -> 56.5 mm, vias 1 -> 2
- net SOIL_PWR: track 19.5 -> 50.7 mm, vias 0 -> 1
- net TEMP_DAT: track 21.2 -> 52.2 mm, vias 0 -> 1
- net 3.3V: track 120.8 -> 149.9 mm, vias 1 -> 5
- net SDA: track 4.79 -> 30.3 mm, vias 0 -> 2
- net SCL: track 10.5 -> 32.3 mm, vias 0 -> 2
- net N$14: track 0.00 -> 20.0 mm
- net 3: track 17.8 -> 0.00 mm
- net 7: track 17.4 -> 0.00 mm
- net 9: track 15.6 -> 0.00 mm
- net N$7: track 0.00 -> 15.5 mm
- net 11: track 14.5 -> 0.00 mm
- net N$11: track 3.35 -> 17.7 mm, vias 0 -> 1
- net 15: track 13.3 -> 0.00 mm
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Other:
- board size 68.6 x 63.5 mm -> 68.6 x 58.4 mm

Commit message: Updated brd and sch file 3/28/2017
Parts:
- removed R2, R3: 4.7k, SparkFun-Resistors:0603
- added I2C: JUMPER-SMT_3_2-NC_TRACE_SILK, SparkFun-Jumpers:SMT-JUMPER_3_2-NC_TRACE_SILK
- added J8, J9: (no value), SparkFun-Connectors:1X04
- added R12, R13: 4.7k, SparkFun-Resistors:0603
- moved LOGO4 50.6 mm to (66.4, 54.0)
- moved LOGO1 46.7 mm to (43.5, 36.5)
- moved R1 15.2 mm to (29.2, 21.6)
- moved C1 7.10 mm to (31.8, 37.5)
- moved C2 7.10 mm to (36.8, 37.5)
- moved U1 7.10 mm to (34.3, 37.5)
- moved R5 1.91 mm to (60.3, 22.9)
- moved R6 1.27 mm to (24.1, 21.6)
- moved R7 1.27 mm to (26.7, 21.6)
- moved D2 1.27 mm to (57.1, 22.9)
- moved D6 0.64 mm to (38.1, 21.0)
- moved R4 0.63 mm to (54.0, 22.9)
Connections:
- removed net 14: J1.A17
- removed net 15: J1.A16
- new net N$4: I2C.3, R12.2
- new net N$8: I2C.1, R13.2
- new net RXI: J1.A17, J8.2
- new net TXO: J1.A16, J8.1
- net 3.3V: now also I2C.2, J8.4, J9.3; no longer R2.2, R3.2
- net GND: now also J8.3, J9.4
- net SCL: now also J9.1, R13.1; no longer R3.1
- net SDA: now also J9.2, R12.1; no longer R2.1
Routing:
- net TXO: track 0.00 -> 49.7 mm
- net RXI: track 0.00 -> 46.8 mm
- net 3.3V: track 149.9 -> 187.0 mm
- net SCL: track 32.3 -> 57.0 mm, vias 2 -> 1
- net SDA: track 30.3 -> 47.7 mm, vias 2 -> 0
- net N$2: track 9.20 -> 23.4 mm, vias 0 -> 2
- net GND: track 11.8 -> 0.00 mm, vias 17 -> 11
- net N$7: track 15.5 -> 7.45 mm
- net N$11: track 17.7 -> 11.9 mm
- net TEMP_DAT: track 52.2 -> 57.8 mm
- net N$8: track 0.00 -> 5.15 mm
- net N$4: track 0.00 -> 5.15 mm
- net SOIL_PWR: track 50.7 -> 55.2 mm
- net N$14: track 20.0 -> 15.9 mm, vias 0 -> 1
- net SOIL_DAT: track 56.5 -> 59.6 mm, vias 2 -> 1
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Other:
- board text added: "GND"
- board text added: "I2C"
- board text added: "I2C PORT"
- board text added: "RAIN"
- board text added: "RX-I"
- board text added: "SCL"
- board text added: "SDA"
- board text added: "SOIL MOISTURE"
- board text added: "SOIL TEMP"
- board text added: "TX-0"
- board text added: "UART SERIAL"
- board text added: "VCC"
- board text added: "WIND"
- board text added: "altitude"
- board text added: "humidity"
- board text added: "pressure"
- board text added: "temp"

Commit message: updated board and sch files 3/29
Parts:
- moved LOGO1 1.16 mm to (42.4, 36.2)
Routing:
- net 3.3V: track 187.0 -> 186.0 mm
Other:
- board text added: "0"
- board text added: "12"
- board text added: "16"
Changed lines of the file:
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@@
 <setting verticaltext="up"/>
 </settings>
-<grid distance="0.0125" unitdist="inch" unit="inch" style="dots" multiple="1" display="yes" altdistance="0.025" altunitdist="inch" altunit="inch"/>
+<grid distance="0.00625" unitdist="inch" unit="inch" style="dots" multiple="1" display="yes" altdistance="0.025" altunitdist="inch" altunit="inch"/>
 <layers>
 <layer number="1" name="Top" color="4" fill="1" visible="yes" active="yes"/>
@@
 <text x="62.23" y="49.53" size="1.778" layer="16" font="vector" ratio="15" rot="SMR270" align="center">v01</text>
 <text x="34.29" y="59.055" size="1.143" layer="22" font="vector" ratio="18" rot="MR0" align="center">weather:bit</text>
-<text x="-30.48" y="35.56" size="1.778" layer="47" font="vector" ratio="15">* All dimensions
+<text x="30.63875" y="90.4875" size="1.778" layer="47" font="vector" ratio="15">* All dimensions
   are in inches</text>
 <wire x1="2.54" y1="63.5" x2="66.04" y2="63.5" width="0.2032" layer="20"/>
@@
 <dimension x1="68.58" y1="5.08" x2="68.58" y2="63.5" x3="85.09" y3="34.29" textsize="1.778" layer="47" unit="inch"/>
 <dimension x1="68.58" y1="63.5" x2="0" y2="63.5" x3="34.29" y3="80.01" textsize="1.778" layer="47" unit="inch"/>
-<text x="56.515" y="33.02" size="1.016" layer="21" font="vector" ratio="15" rot="R90">I2C</text>
-<text x="3.175" y="37.465" size="1.778" layer="21">VCC</text>
-<text x="3.175" y="34.925" size="1.778" layer="21">GND</text>
-<text x="3.175" y="32.385" size="1.778" layer="21">RX-I</text>
-<text x="3.175" y="29.845" size="1.778" layer="21">TX-0</text>
-<text x="65.405" y="38.735" size="1.778" layer="21" rot="R180">GND</text>
-<text x="65.405" y="36.195" size="1.778" layer="21" rot="R180">VCC</text>
-<text x="65.405" y="33.655" size="1.778" layer="21" rot="R180">SDA</text>
-<text x="65.405" y="31.115" size="1.778" layer="21" rot="R180">SCL</text>
-<text x="0" y="40.64" size="1.778" layer="21">UART
+<text x="56.8325" y="33.02" size="1.016" layer="21" font="vector" ratio="15" rot="R90">I2C</text>
+<text x="3.175" y="37.465" size="1.778" layer="21" font="vector" ratio="15">VCC</text>
+<text x="3.175" y="34.925" size="1.778" layer="21" font="vector" ratio="15">GND</text>
+<text x="3.175" y="32.385" size="1.778" layer="21" font="vector" ratio="15">RX-I</text>
+<text x="3.175" y="29.845" size="1.778" layer="21" font="vector" ratio="15">TX-0</text>
+<text x="65.405" y="38.735" size="1.778" layer="21" font="vector" ratio="15" rot="R180">GND</text>
+<text x="65.405" y="36.195" size="1.778" layer="21" font="vector" ratio="15" rot="R180">VCC</text>
+<text x="65.405" y="33.655" size="1.778" layer="21" font="vector" ratio="15" rot="R180">SDA</text>
+<text x="65.405" y="31.115" size="1.778" layer="21" font="vector" ratio="15" rot="R180">SCL</text>
+<text x="0.15875" y="40.9575" size="1.778" layer="21" font="vector" ratio="15">UART
 SERIAL</text>
-<text x="62.865" y="40.64" size="1.778" layer="21">I2C
+<text x="62.07125" y="40.64" size="1.778" layer="21" font="vector" ratio="15">I2C
 PORT</text>
-<text x="38.735" y="24.13" size="1.778" layer="21">SOIL
+<text x="41.275" y="28.41625" size="1.778" layer="21" font="vector" ratio="15" align="top-center">SOIL
 TEMP</text>
-<text x="20.32" y="24.13" size="1.778" layer="21">    SOIL
+<text x="26.67" y="28.575" size="1.778" layer="21" font="vector" ratio="15" align="top-center">SOIL
 MOISTURE</text>
-<wire x1="29.845" y1="41.275" x2="29.845" y2="33.655" width="0.254" layer="21"/>
-<wire x1="29.845" y1="33.655" x2="38.735" y2="33.655" width="0.254" layer="21"/>
-<wire x1="38.735" y1="33.655" x2="38.735" y2="41.275" width="0.254" layer="21"/>
-<wire x1="38.735" y1="41.275" x2="29.845" y2="41.275" width="0.254" layer="21"/>
-<text x="29.845" y="42.545" size="1.778" layer="21">humidity</text>
-<text x="41.275" y="32.385" size="1.778" layer="21" rot="R90">pressure</text>
-<text x="28.575" y="34.925" size="1.778" layer="21" rot="R90">temp</text>
-<text x="30.48" y="31.115" size="1.778" layer="21">altitude</text>
+<wire x1="30.48" y1="40.005" x2="30.48" y2="34.925" width="0.254" layer="21"/>
+<wire x1="30.48" y1="34.925" x2="38.1" y2="34.925" width="0.254" layer="21"/>
+<wire x1="38.1" y1="34.925" x2="38.1" y2="40.005" width="0.254" layer="21"/>
+<wire x1="38.1" y1="40.005" x2="30.48" y2="40.005" width="0.254" layer="21"/>
+<text x="30.48" y="40.64" size="1.27" layer="21" font="vector" ratio="15">humidity</text>
+<text x="39.6875" y="33.02" size="1.27" layer="21" font="vector" ratio="15" rot="R90">pressure</text>
+<text x="29.845" y="35.56" size="1.27" layer="21" font="vector" ratio="15" rot="R90">temp</text>
+<text x="30.48" y="33.02" size="1.27" layer="21" font="vector" ratio="15">altitude</text>
 <wire x1="20.955" y1="23.495" x2="31.115" y2="23.495" width="0.254" layer="21"/>
 <wire x1="31.115" y1="23.495" x2="33.02" y2="21.59" width="0.254" layer="21" curve="-90"/>
@@
 <wire x1="36.195" y1="6.35" x2="38.1" y2="6.35" width="0.254" layer="21"/>
 <text x="8.255" y="25.4" size="1.778" layer="21" font="vector" ratio="15">WIND</text>
-<text x="52.705" y="25.4" size="1.778" layer="21">RAIN</text>
-<text x="9.525" y="31.115" size="2.1844" layer="21" font="vector" ratio="15">weather:bit</text>
+<text x="52.705" y="25.4" size="1.778" layer="21" font="vector" ratio="15">RAIN</text>
+<text x="9.525" y="36.67125" size="2.1844" layer="21" font="vector" ratio="20">weather:bit</text>
+<text x="23.1775" y="8.255" size="1.016" layer="21" font="vector" ratio="15">16</text>
+<text x="25.7175" y="8.255" size="0.889" layer="21" font="vector" ratio="15">GND</text>
+<text x="28.8925" y="8.255" size="1.016" layer="21" font="vector" ratio="15">0</text>
+<text x="38.1" y="8.255" size="0.889" layer="21" font="vector" ratio="15">VCC</text>
+<text x="41.11625" y="8.255" size="1.016" layer="21" font="vector" ratio="15">12</text>
+<text x="43.815" y="8.255" size="0.889" layer="21" font="vector" ratio="15">GND</text>
+<dimension x1="2.54" y1="60.96" x2="66.04" y2="60.96" x3="34.29" y3="73.9775" textsize="1.016" layer="47" unit="inch"/>
+<dimension x1="66.04" y1="60.96" x2="66.04" y2="7.62" x3="79.21625" y3="34.29" textsize="1.016" layer="47" unit="inch"/>
 </plain>
 <attributes>
@@
 <attribute name="PROD_ID" value="RES-07857" x="45.085" y="21.59" size="1.778" layer="27" rot="R270" display="off"/>
 </element>
-<element name="LOGO1" library="SparkFun-Aesthetics" package="SFE_LOGO_NAME_FLAME_.1" value="SFE_LOGO_NAME_FLAME.1_INCH" x="43.4975" y="36.5125"/>
+<element name="LOGO1" library="SparkFun-Aesthetics" package="SFE_LOGO_NAME_FLAME_.1" value="SFE_LOGO_NAME_FLAME.1_INCH" x="42.38625" y="36.195"/>
 <element name="LOGO4" library="SparkFun-Aesthetics" package="OSHW-LOGO-S" value="OSHW-LOGOS" x="66.3575" y="53.975"/>
 <element name="H3" library="SparkFun-Electromechanical" package="STAND-OFF" value="STAND-OFF" x="2.54" y="7.62"/>
@@
 <via x="34.925" y="8.255" extent="1-16" drill="0.635"/>
 <via x="55.245" y="40.9575" extent="1-16" drill="0.635"/>
-<via x="41.91" y="43.4975" extent="1-16" drill="0.635"/>
+<via x="41.275" y="45.085" extent="1-16" drill="0.635"/>
 <contactref element="J8" pad="3"/>
 <contactref element="J9" pad="4"/>
-<via x="63.1825" y="33.02" extent="1-16" drill="0.635"/>
 <via x="60.325" y="36.195" extent="1-16" drill="0.635"/>
-<via x="20.6375" y="42.545" extent="1-16" drill="0.635"/>
+<via x="28.575" y="42.8625" extent="1-16" drill="0.635"/>
 </signal>
 <signal name="3.3V">
@@
 <wire x1="37.9222" y1="15.24" x2="37.9222" y2="7.7978" width="0.254" layer="1"/>
 <wire x1="37.9222" y1="7.7978" x2="39.37" y2="6.35" width="0.254" layer="1"/>
-<via x="10.795" y="20.32" extent="1-16" drill="0.381"/>
-<via x="6.35" y="20.32" extent="1-16" drill="0.381"/>
+<via x="10.795" y="20.32" extent="1-16" drill="0.635"/>
+<via x="6.35" y="20.32" extent="1-16" drill="0.635"/>
 <wire x1="6.35" y1="20.32" x2="6.35" y2="21.71" width="0.254" layer="1"/>
 <wire x1="10.795" y1="20.32" x2="11.43" y2="20.32" width="0.254" layer="1"/>
@@
 <wire x1="67.31" y1="35.56" x2="61.2775" y2="35.56" width="0.254" layer="16"/>
 <wire x1="61.2775" y1="35.56" x2="60.0075" y2="34.29" width="0.254" layer="16"/>
-<wire x1="58.1025" y1="33.274" x2="58.1025" y2="34.29" width="0.254" layer="1"/>
-<wire x1="58.1025" y1="34.29" x2="54.9275" y2="34.29" width="0.254" layer="1"/>
-<via x="54.9275" y="34.29" extent="1-16" drill="0.635"/>
-<wire x1="54.9275" y1="34.29" x2="44.45" y2="34.29" width="0.254" layer="16"/>
+<wire x1="58.1025" y1="34.29" x2="54.2925" y2="34.29" width="0.254" layer="1"/>
+<via x="54.2925" y="34.29" extent="1-16" drill="0.635"/>
+<wire x1="54.2925" y1="34.29" x2="44.45" y2="34.29" width="0.254" layer="16"/>
 <wire x1="44.45" y1="34.29" x2="43.815" y2="34.925" width="0.254" layer="16"/>
 </signal>
@@
 </signal>
 </signals>
+<errors>
+</errors>
 </board>
 </drawing>

Commit message: Adding Library Part Updated Brd File Updated Sch File 3/30/2017
Parts:
- removed I2C: JUMPER-SMT_3_2-NC_TRACE_SILK, SparkFun-Jumpers:SMT-JUMPER_3_2-NC_TRACE_SILK
- removed J1: EDGE-80PTH-RA, local_lib:VEC-127-080-R
- removed R12, R13: 4.7k, SparkFun-Resistors:0603
- added U2: micro:bit, Micro_Bit_Parts:MICRO:BIT_RA_PTH
- LOGO2: value SFE_LOGO_NAME_FLAME.1_INCH -> SFE_LOGO_NAME_FLAME.3_INCH; device SparkFun-Aesthetics:SFE_LOGO_NAME_FLAME_.1 -> SparkFun-Aesthetics:SFE_LOGO_NAME_FLAME_.3
- LOGO3, LOGO4: value OSHW-LOGOS -> OSHW-LOGOL; device SparkFun-Aesthetics:OSHW-LOGO-S -> SparkFun-Aesthetics:OSHW-LOGO-L
- moved FD4 76.1 mm to (67.2, 11.4)
- moved FD3 60.3 mm to (1.71, 56.3)
- moved FD1 50.7 mm to (2.57, 12.0)
- moved LOGO3 41.7 mm to (34.0, 23.8)
- moved LOGO1 28.2 mm to (14.3, 38.9)
- moved LOGO2 27.5 mm to (50.6, 31.4)
- moved LOGO4 21.2 mm to (52.5, 37.9)
- moved FD2 4.94 mm to (66.9, 47.5)
- moved C2 4.15 mm to (41.0, 37.9)
- moved C1 4.15 mm to (35.9, 37.9)
- moved U1 4.15 mm to (38.4, 37.9)
- moved R7 0.64 mm to (26.0, 21.6)
- moved R6 0.63 mm to (23.5, 21.6)
Connections:
- removed net N$4: I2C.3, R12.2
- removed net N$8: I2C.1, R13.2
- net 10: now also U2.A25; no longer J1.A25
- net 11: now also U2.A24; no longer J1.A24
- net 13: now also U2.A18; no longer J1.A18
- net 3: now also U2.A40; no longer J1.A40
- net 3.3V: now also U2.A10, U2.A11, U2.A12, U2.A13, U2.A14, U2.A9; no longer I2C.2, J1.A10, J1.A11, J1.A12, J1.A13, J1.A14, J1.A9
- net 4: now also U2.A35; no longer J1.A35
- net 5: now also U2.A34; no longer J1.A34
- net 6: now also U2.A33; no longer J1.A33
- net 7: now also U2.A32; no longer J1.A32
- net 9: now also U2.A26; no longer J1.A26
- net GND: now also U2.A1, U2.A2, U2.A3, U2.A4, U2.A5, U2.A6; no longer J1.A1, J1.A2, J1.A3, J1.A4, J1.A5, J1.A6
- net RAIN: now also U2.A19, U2.A20, U2.A21, U2.A22; no longer J1.A19, J1.A20, J1.A21, J1.A22
- net RXI: now also U2.A17; no longer J1.A17
- net SCL: now also U2.A8; no longer J1.A8, R13.1
- net SDA: now also U2.A7; no longer J1.A7, R12.1
- net SOIL_DAT: now also U2.A36, U2.A37, U2.A38, U2.A39; no longer J1.A36, J1.A37, J1.A38, J1.A39
- net SOIL_PWR: now also U2.A15; no longer J1.A15
- net TEMP_DAT: now also U2.A23; no longer J1.A23
- net TXO: now also U2.A16; no longer J1.A16
- net WDIR: now also U2.A28, U2.A29, U2.A30, U2.A31; no longer J1.A28, J1.A29, J1.A30, J1.A31
- net WSPEED: now also U2.A27; no longer J1.A27
Routing:
- net WDIR: track 69.2 -> 46.7 mm, vias 1 -> 2
- net SCL: track 57.0 -> 43.9 mm
- net SDA: track 47.7 -> 40.2 mm
- net N$8: track 5.15 -> 0.00 mm
- net N$4: track 5.15 -> 0.00 mm
- net SOIL_DAT: track 59.6 -> 64.1 mm
- net N$2: track 23.4 -> 27.0 mm
- net 3.3V: track 186.0 -> 189.0 mm, vias 5 -> 3
- net N$14: track 15.9 -> 18.1 mm
- net SOIL_PWR: track 55.2 -> 56.1 mm
- net N$13: track 10.4 -> 9.59 mm
Other:
- board text added: "RXI"
- board text added: "TXO"
- board text removed: "I2C"
- board text removed: "RX-I"
- board text removed: "TX-0"

Commit message: Updated BRD and SCH files per Design Review 3/31
Parts:
- moved H3 5.08 mm to (2.54, 2.54)
- moved H4 5.08 mm to (66.0, 2.54)
- moved H1 3.81 mm to (2.54, 64.8)
- moved H2 3.81 mm to (66.0, 64.8)
- moved LOGO1 3.27 mm to (15.1, 35.7)
- moved LOGO2 2.54 mm to (50.6, 28.9)
- moved FD1 2.54 mm to (2.57, 9.46)
- moved J4 2.54 mm to (38.1, 12.7)
- moved J5 2.54 mm to (22.9, 12.7)
- moved J2 2.54 mm to (55.9, 7.62)
- moved J3 2.54 mm to (12.7, 7.62)
- moved J6 2.54 mm to (39.4, 3.81)
- moved J7 2.54 mm to (24.1, 3.81)
- moved C1 2.54 mm to (35.9, 35.4)
- moved C2 2.54 mm to (41.0, 35.4)
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Routing:
- net TEMP_DAT: track 57.9 -> 59.8 mm
- net RAIN: track 48.6 -> 49.3 mm
Other:
- board size 68.6 x 58.4 mm -> 68.6 x 67.3 mm
- board text added: "Mary West, based on Weather Shield Design by Nathan Siedle"
- board text added: "P0"
- board text added: "P12"
- board text added: "P16"
- board text added: "SERIAL PORT(GPS)"
- board text added: "SIG"
- board text added: "alt"
- board text removed: "0"
- board text removed: "12"
- board text removed: "16"
- board text removed: "Mary West"
- board text removed: "UART SERIAL"
- board text removed: "altitude"
