File: Hardware/weather-bit.brd (EAGLE design)
At the start: 68.6 x 58.4 mm, 74 parts, among them J10 SMD, J2 RJ11, J3 RJ11, J6 455-1750-1-ND, J7 455-1750-1-ND, J8 Qwiic (vertical), J9 SMD, U1 BME280, U2 micro:bit

Commit message: sch cleanup and move to one sheet
Parts:
- removed FRAME2: FRAME-LETTER, SparkFun-Aesthetics:CREATIVE_COMMONS
- J6, J7: value 455-1750-1-ND -> (none)
Other:
- board text added: "Pete Lewis"
- board text added: "Revised by:"
Changed lines of the file:
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@@
 <board>
 <plain>
-<text x="31.75" y="-11.43" size="1.778" layer="51" font="vector" ratio="15">Mary West, based on Weather Shield Design by Nathan Seidle </text>
+<text x="31.75" y="-11.43" size="1.778" layer="51" font="vector" ratio="9">Mary West, based on Weather Shield Design by Nathan Seidle </text>
 <text x="67.16395" y="18.07845" size="1.778" layer="16" font="vector" ratio="15" rot="SMR270" align="center">v11</text>
 <text x="30.63875" y="90.4875" size="1.778" layer="47" font="vector" ratio="15">* All dimensions
@@
 <dimension x1="2.54" y1="64.77" x2="0.79375" y2="64.77" x3="1.666875" y3="69.5325" textsize="1.778" layer="47" unit="inch"/>
 <text x="6.223" y="-32.385" size="2.54" layer="51">Solder Mask: Black Gloss</text>
+<text x="11.43" y="-13.97" size="1.778" layer="51" font="vector">Revised by:</text>
+<text x="29.21" y="-13.97" size="1.778" layer="51" font="vector">Pete Lewis</text>
 </plain>
 <attributes>
@@
 <element name="FD3" library="SparkFun-Aesthetics" package="FIDUCIAL-1X2" value="FIDUCIAL1X2" x="1.7145" y="44.86275" smashed="yes" rot="MR0"/>
 <element name="FD4" library="SparkFun-Aesthetics" package="FIDUCIAL-1X2" value="FIDUCIAL1X2" x="67.183" y="8.89" smashed="yes" rot="MR0"/>
-<element name="FRAME2" library="SparkFun-Aesthetics" package="CREATIVE_COMMONS" value="FRAME-LETTER" x="0" y="-11.43" smashed="yes"/>
 <element name="U1" library="SparkFun-Sensors" package="LGA-8-2.5X2.5" value="BME280" x="47.16145" y="33.9852" smashed="yes">
 <attribute name="NAME" x="45.89145" y="35.5092" size="0.6096" layer="25" font="vector" ratio="20"/>
@@
 <attribute name="VALUE" x="24.765" y="8.001" size="0.6096" layer="27" font="vector" ratio="20"/>
 </element>
-<element name="J6" library="SparkFun-Connectors" package="1X03" value="455-1750-1-ND" x="39.37" y="3.81" smashed="yes">
+<element name="J6" library="SparkFun-Connectors" package="1X03" value="" x="39.37" y="3.81" smashed="yes">
 <attribute name="NAME" x="38.1" y="5.207" size="0.6096" layer="25" font="vector" ratio="20"/>
 <attribute name="PROD_ID" value="XXX-00000" x="39.37" y="3.81" size="1.778" layer="27" display="off"/>
 <attribute name="VALUE" value="455-1750-1-ND" x="38.1" y="1.778" size="0.6096" layer="27" font="vector" ratio="20"/>
 </element>
-<element name="J7" library="SparkFun-Connectors" package="1X03" value="455-1750-1-ND" x="24.13" y="3.81" smashed="yes">
+<element name="J7" library="SparkFun-Connectors" package="1X03" value="" x="24.13" y="3.81" smashed="yes">
 <attribute name="NAME" x="22.86" y="5.207" size="0.6096" layer="25" font="vector" ratio="20"/>
 <attribute name="PROD_ID" value="XXX-00000" x="24.13" y="3.81" size="1.778" layer="27" display="off"/>
